Commit message: feat: update to jazzy moveit; had to add accel limits

File: src/arm_moveit_config/config/for.ros2_control.xacro (robot description, xacro)
@@ -2,5 +2,5 @@
 <robot xmlns:xacro="http://www.ros.org/wiki/xacro">
     <xacro:macro name="for_ros2_control" params="name initial_positions_file">
-        <xacro:property name="initial_positions" value="${load_yaml(initial_positions_file)['initial_positions']}"/>
+        <xacro:property name="initial_positions" value="${xacro.load_yaml(initial_positions_file)['initial_positions']}"/>
         <ros2_control name="${name}" type="system">
             <hardware>

Commit message: feat: build topic_based_ros2_control from source to use PR that waits for initial state

File: src/arm_moveit_config/config/for.ros2_control.xacro (robot description, xacro)
@@ -1,6 +1,7 @@
 <?xml version="1.0"?>
 <robot xmlns:xacro="http://www.ros.org/wiki/xacro">
-    <xacro:macro name="for_ros2_control" params="name initial_positions_file">
-        <xacro:property name="initial_positions" value="${xacro.load_yaml(initial_positions_file)['initial_positions']}"/>
+    <!-- <xacro:macro name="for_ros2_control" params="name initial_positions_file"> -->
+    <xacro:macro name="for_ros2_control" params="name">
+        <!-- <xacro:property name="initial_positions" value="${xacro.load_yaml(initial_positions_file)['initial_positions']}"/> -->
         <ros2_control name="${name}" type="system">
             <hardware>
@@ -10,10 +11,11 @@
                 <plugin>topic_based_ros2_control/TopicBasedSystem</plugin>
                 <param name="trigger_joint_command_threshold">0.001</param>
-                <param name="sum_wrapped_joint_states">true</param>
+                <param name="sum_wrapped_joint_states">false</param>
+                <param name="use_initial_states_as_initial_commands">true</param>
             </hardware>
             <joint name="base_revolute">
                 <command_interface name="position"/>
                 <state_interface name="position">
-                  <param name="initial_value">${initial_positions['base_revolute']}</param>
+                  <!-- <param name="initial_value">${initial_positions['base_revolute']}</param> -->
                 </state_interface>
             </joint>
@@ -21,5 +23,5 @@
                 <command_interface name="position"/>
                 <state_interface name="position">
-                  <param name="initial_value">${initial_positions['double_revolute_1']}</param>
+                  <!-- <param name="initial_value">${initial_positions['double_revolute_1']}</param> -->
                 </state_interface>
             </joint>
@@ -27,5 +29,5 @@
                 <command_interface name="position"/>
                 <state_interface name="position">
-                  <param name="initial_value">${initial_positions['double_spin']}</param>
+                  <!-- <param name="initial_value">${initial_positions['double_spin']}</param> -->
                 </state_interface>
             </joint>
@@ -33,5 +35,5 @@
                 <command_interface name="position"/>
                 <state_interface name="position">
-                  <param name="initial_value">${initial_positions['double_revolute_2']}</param>
+                  <!-- <param name="initial_value">${initial_positions['double_revolute_2']}</param> -->
                 </state_interface>
             </joint>
@@ -39,5 +41,5 @@
                 <command_interface name="position"/>
                 <state_interface name="position">
-                  <param name="initial_value">${initial_positions['middle_revolute']}</param>
+                  <!-- <param name="initial_value">${initial_positions['middle_revolute']}</param> -->
                 </state_interface>
             </joint>
@@ -45,5 +47,5 @@
                 <command_interface name="position"/>
                 <state_interface name="position">
-                  <param name="initial_value">${initial_positions['middle_spin']}</param>
+                  <!-- <param name="initial_value">${initial_positions['middle_spin']}</param> -->
                 </state_interface>
             </joint>
@@ -51,5 +53,5 @@
                 <command_interface name="position"/>
                 <state_interface name="position">
-                  <param name="initial_value">${initial_positions['end_revolute_1']}</param>
+                  <!-- <param name="initial_value">${initial_positions['end_revolute_1']}</param> -->
                 </state_interface>
             </joint>
@@ -57,5 +59,5 @@
                 <command_interface name="position"/>
                 <state_interface name="position">
-                  <param name="initial_value">${initial_positions['end_revolute_2']}</param>
+                  <!-- <param name="initial_value">${initial_positions['end_revolute_2']}</param> -->
                 </state_interface>
             </joint>
@@ -63,5 +65,5 @@
                 <command_interface name="position"/>
                 <state_interface name="position">
-                  <param name="initial_value">${initial_positions['effector_spin']}</param>
+                  <!-- <param name="initial_value">${initial_positions['effector_spin']}</param> -->
                 </state_interface>
             </joint>

File: src/arm_moveit_config/config/for.urdf.xacro (robot description, xacro)
@@ -1,9 +1,10 @@
 <?xml version="1.0"?>
 <robot xmlns:xacro="http://www.ros.org/wiki/xacro" name="for">
-    <xacro:arg name="initial_positions_file" default="initial_positions.yaml" />
+    <!-- <xacro:arg name="initial_positions_file" default="initial_positions.yaml" /> -->
     <!-- Import for urdf file -->
     <xacro:include filename="$(find arm_description)/urdf/model.urdf" />
     <!-- Import control_xacro -->
     <xacro:include filename="for.ros2_control.xacro" />
-    <xacro:for_ros2_control name="FakeSystem" initial_positions_file="$(arg initial_positions_file)"/>
+    <!-- <xacro:for_ros2_control name="FakeSystem" initial_positions_file="$(arg initial_positions_file)"/> -->
+    <xacro:for_ros2_control name="FakeSystem" />
 </robot>
